File: Board1/TheHub.sch (KiCad schematic (older format))
At the start: 43 parts, among them J1 Actuator Fdbk Conn, J11 RFD900, J12 I2C_1 Test Point, J13 I2C_2 Test Point, J15 GPIO Test, J16 I2C_3 Test Point, J17 12V OUT, J18 7.4V IN, J2 QuadEnc_Conn, J23 NucleoRight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

Commit message: Update netlist to use staight headars instead of angled
Parts:
- J1: footprint Pin_Headers:Pin_Header_Angled_2x03_Pitch2.54mm -> Pin_Headers:Pin_Header_Straight_2x03_Pitch2.54mm
- J2: footprint Pin_Headers:Pin_Header_Angled_1x04_Pitch2.54mm -> Pin_Headers:Pin_Header_Straight_1x04_Pitch2.54mm
Changed lines of the file:
@@
 F 0 "J1" H 7800 4000 50  0000 C CNN
 F 1 "Actuator Fdbk Conn" H 7800 3450 50  0000 C CNN
-F 2 "Pin_Headers:Pin_Header_Angled_2x03_Pitch2.54mm" H 7750 3800 50  0001 C CNN
+F 2 "Pin_Headers:Pin_Header_Straight_2x03_Pitch2.54mm" H 7750 3800 50  0001 C CNN
 F 3 "" H 7750 3800 50  0001 C CNN
 	1    7750 3800
@@
 F 0 "J2" H 9350 4600 50  0000 C CNN
 F 1 "QuadEnc_Conn" H 9350 4100 50  0000 C CNN
-F 2 "Pin_Headers:Pin_Header_Angled_1x04_Pitch2.54mm" H 9350 4400 50  0001 C CNN
+F 2 "Pin_Headers:Pin_Header_Straight_1x04_Pitch2.54mm" H 9350 4400 50  0001 C CNN
 F 3 "" H 9350 4400 50  0001 C CNN
 	1    9350 4400
