File: Board1/TheHub.kicad_pcb (KiCad board)
At the start: 2 copper layers, 118.7 x 184.1 mm, 59 parts, among them J1 Actuator Fdbk Conn, J11 RFD900, J12 I2C_1 Test Point, J13 I2C_2 Test Point, J15 GPIO Test, J16 I2C_3 Test Point, J17 12V OUT, J2 QuadEnc_Conn, J23 NucleoRight, J5 NucleoLeft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

Commit message: Add BOM
Other:
- board text added: "Analog Feedback"
- board text added: "PC0"
- board text added: "PC1"
- board text removed: "A_Fdbk PC0"
- board text removed: "A_Fdbk PC1"
Changed lines of the file:
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@@
     (links 114)
     (no_connects 1)
-    (area 62.154999 50.724999 181.050001 235.025001)
+    (area 56.482857 49.435 186.087143 236.415)
     (thickness 1.6)
-    (drawings 68)
+    (drawings 69)
     (tracks 429)
     (zones 0)
@@
     (pad "" thru_hole circle (at 0 -12.7 180) (size 3.302 3.302) (drill 2.54) (layers *.Cu *.Mask))
   )
+  (gr_text "Analog\nFeedback" (at 67.056 162.56) (layer F.SilkS)
+    (effects (font (size 1 1) (thickness 0.15)))
+  )
   (gr_text "PA2 TX2" (at 133.35 168.656) (layer F.SilkS)
     (effects (font (size 1 1) (thickness 0.15)))
@@
     (effects (font (size 1 1) (thickness 0.15)))
   )
-  (gr_text "A_Fdbk PC0" (at 67.818 162.814 90) (layer F.SilkS)
+  (gr_text PC0 (at 68.072 165.608 90) (layer F.SilkS)
     (effects (font (size 1 1) (thickness 0.15)))
   )
-  (gr_text "A_Fdbk PC1" (at 65.532 162.814 90) (layer F.SilkS)
+  (gr_text PC1 (at 65.278 165.608 90) (layer F.SilkS)
     (effects (font (size 1 1) (thickness 0.15)))
   )
