File: Board2/TheHub.sch (KiCad schematic (older format))
At the start: 35 parts, among them J1 Actuator Fdbk Conn, J11 RFD900, J12 I2C_1 Test Point, J15 GPIO Test, J17 12V OUT, J8 12V MAIN POWER, U10 ADXL377, U11 BNO055, U12 MPL115A2, U13 GPS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

Commit message: Create footprint for Feather M0, correct schematic changes
Parts:
- removed U?: FeatherM0, symbol FeatherM0
- added U?: FeatherM0, symbol FeatherM0
- R10, R5: renamed from R?; footprint (none) -> Resistors_SMD:R_0805
- gave numbers to parts that had none: 1
Connections:
- net +3V3: now also U?.2 (3.3V)
- net A0: now also U?.5 (A0)
- net A1: now also U?.6 (A1)
- net A2: now also U?.7 (A2)
- net A_FDBK_0: now also U?.8 (A3)
- net A_FDBK_1: now also U?.9 (A4)
- net GND: now also U?.16 (GND), U?.4 (GND)
- net SCL_1: now also U?.18 (SCL)
- net SDA_1: now also U?.17 (SDA)
- net Status1: now also U?.19 (5)
- net Status2: now also U?.21 (9)
- net Status3: now also U?.22 (10)
- net Status4: now also U?.23 (11)
- net at R10.1: now also U?.15 (TX)
- net at R5.1: now also U?.14 (RX)

Commit message: Relayout Hub 2 Board
Parts:
- removed U13: GPS, FoxWestern:Adafruit_GPS, symbol GPS
- added U4: GT-U7_GPS, FoxWestern:GT-U7_GPS, symbol GT-U7_GPS
- U1: renamed from U?; footprint (none) -> FoxWestern:FeatherM0
- U3: footprint (none) -> FoxWestern:ArduinoNano
Connections:
- net +3V3: now also U4.5 (VCC)
- net GND: now also U4.4 (GND)
- net GPS_RX: now also U4.3 (RX)
- net GPS_TX: now also U4.2 (TX)
- net GPS_FIX: no longer names the net of U3.25 (D7)
- no-connect marks 62 -> 60
Other:
- note removed: "GPS_FIX is HIGH when\nthe unit has a GPS lock."
