File: Board3/AvionicsBoard.sch (KiCad schematic (older format))
At the start: 54 parts

Commit message: Associate some arts, make some schematic changes
Parts:
- BT1: renamed from BT?; footprint (none) -> TO_SOT_Packages_SMD:SOT-23-5
- J1: renamed from J?; footprint (none) -> Connectors:USB_Mini-B
- J2: renamed from J?; footprint (none) -> FoxWestern:XT60
- J3: renamed from J?; footprint (none) -> Pin_Headers:Pin_Header_Straight_1x04_Pitch2.54mm
- J4, J5: renamed from J?; footprint (none) -> Pin_Headers:Pin_Header_Straight_1x02_Pitch2.54mm
- J6: renamed from J?; footprint (none) -> Connectors:microSD_Card_Receptacle_Wuerth_693072010801
- J7: renamed from J?; footprint (none) -> Connectors:SMA_SMD_Jack_Straight
- J8: renamed from J?; footprint (none) -> Pin_Headers:Pin_Header_Straight_2x03_Pitch2.54mm
- J9: renamed from J?; footprint (none) -> Pin_Headers:Pin_Header_Straight_2x02_Pitch2.54mm
- U1: renamed from U?; footprint (none) -> TO_SOT_Packages_SMD:SOT-223-3_TabPin2
- U2: renamed from U?; footprint (none) -> Housings_QFP:TQFP-48_7x7mm_Pitch0.5mm
- U3: renamed from U?; footprint (none) -> TO_SOT_Packages_SMD:SOT-23-5
- U6: renamed from U?; footprint (none) -> Housings_LGA:LGA-8_3x5mm_Pitch1.25mm
- U7: renamed from U?; footprint (none) -> FoxWestern:BNO055-LGA
- gave numbers to parts that had none: 39
Connections:
- net D5 is gone; now on net CS: U2.24 (PA15)
Other:
- moved on the sheet: BT1, C1, C10, C11, C12, C13, C14, C15, C16, C17, C18, C19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
