File: Board3/_saved_AvionicsBoard.sch (KiCad schematic (older format))
At the start: 58 parts, among them J1 USB_A, J10 I2C, J11 UART, J2 Conn_01x02, J3 SWD, J4 7.2V, J5 3.3V, J6 Micro_SD_Card, J7 RF IN, J8 FDBK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

Commit message: create more footprints, associate parts
Parts:
- J10, J11: footprint (none) -> Pin_Headers:Pin_Header_Straight_1x03_Pitch2.54mm
- R1, R13, R5, R6: footprint (none) -> Resistors_SMD:R_0603_HandSoldering
- R10, R11, R12, R2, R3, R4, R7, R8, R9: footprint (none) -> Resistors_SMD:R_0805
Connections:
- net +3V3: no longer U8.1 (Vin), U8.2 (GND)
- net CS: no longer U8.8 (CS)
- net MISO: no longer U8.6 (MISO)
- net MOSI: no longer U8.7 (MOSI)
- net SCK: no longer U8.5 (SCK)
Other:
- moved on the sheet: U8
Changed lines of the file:
@@
 L RFM95W U8
 U 1 1 5B1B73E9
-P 4150 10100
-F 0 "U8" H 4400 9850 60  0000 C CNN
-F 1 "RFM95W" H 4200 10850 60  0000 C CNN
-F 2 "" H 4150 10100 60  0001 C CNN
-F 3 "" H 4150 10100 60  0001 C CNN
-	1    4150 10100
+P 2300 10200
+F 0 "U8" H 2550 9950 60  0000 C CNN
+F 1 "RFM95W" H 2350 10950 60  0000 C CNN
+F 2 "" H 2300 10200 60  0001 C CNN
+F 3 "" H 2300 10200 60  0001 C CNN
+	1    2300 10200
 	1    0    0    -1
 $EndComp
@@
 F 0 "R10" V 5030 6600 50  0000 C CNN
 F 1 "10k" V 4950 6600 50  0000 C CNN
-F 2 "" V 4880 6600 50  0001 C CNN
+F 2 "Resistors_SMD:R_0805" V 4880 6600 50  0001 C CNN
 F 3 "" H 4950 6600 50  0001 C CNN
 	1    4950 6600
@@
 F 0 "R11" V 6380 7800 50  0000 C CNN
 F 1 "10k" V 6300 7800 50  0000 C CNN
-F 2 "" V 6230 7800 50  0001 C CNN
+F 2 "Resistors_SMD:R_0805" V 6230 7800 50  0001 C CNN
 F 3 "" H 6300 7800 50  0001 C CNN
 	1    6300 7800
@@
 F 0 "R12" V 7480 6850 50  0000 C CNN
 F 1 "10k" V 7400 6850 50  0000 C CNN
-F 2 "" V 7330 6850 50  0001 C CNN
+F 2 "Resistors_SMD:R_0805" V 7330 6850 50  0001 C CNN
 F 3 "" H 7400 6850 50  0001 C CNN
 	1    7400 6850
@@
 F 0 "R2" V 2980 4250 50  0000 C CNN
 F 1 "2.2k" V 2900 4250 50  0000 C CNN
-F 2 "" V 2830 4250 50  0001 C CNN
+F 2 "Resistors_SMD:R_0805" V 2830 4250 50  0001 C CNN
 F 3 "" H 2900 4250 50  0001 C CNN
 	1    2900 4250
@@
 F 0 "R3" V 3230 4250 50  0000 C CNN
 F 1 "2.2k" V 3150 4250 50  0000 C CNN
-F 2 "" V 3080 4250 50  0001 C CNN
+F 2 "Resistors_SMD:R_0805" V 3080 4250 50  0001 C CNN
 F 3 "" H 3150 4250 50  0001 C CNN
 	1    3150 4250
@@
 F 0 "R9" V 7730 2700 50  0000 C CNN
 F 1 "10K" V 7650 2700 50  0000 C CNN
-F 2 "" V 7580 2700 50  0001 C CNN
+F 2 "Resistors_SMD:R_0805" V 7580 2700 50  0001 C CNN
 F 3 "" H 7650 2700 50  0001 C CNN
 	1    7650 2700
@@
 F 0 "R7" V 6080 3750 50  0000 C CNN
 F 1 "10K" V 6000 3750 50  0000 C CNN
-F 2 "" V 5930 3750 50  0001 C CNN
+F 2 "Resistors_SMD:R_0805" V 5930 3750 50  0001 C CNN
 F 3 "" H 6000 3750 50  0001 C CNN
 	1    6000 3750
@@
 F 0 "R8" V 6080 3950 50  0000 C CNN
 F 1 "10K" V 6000 3950 50  0000 C CNN
-F 2 "" V 5930 3950 50  0001 C CNN
+F 2 "Resistors_SMD:R_0805" V 5930 3950 50  0001 C CNN
 F 3 "" H 6000 3950 50  0001 C CNN
 	1    6000 3950
@@
 F 0 "R1" V 1830 2650 50  0000 C CNN
 F 1 "1K" V 1750 2650 50  0000 C CNN
-F 2 "" V 1680 2650 50  0001 C CNN
+F 2 "Resistors_SMD:R_0603_HandSoldering" V 1680 2650 50  0001 C CNN
 F 3 "" H 1750 2650 50  0001 C CNN
 	1    1750 2650
@@
 F 0 "R4" V 3480 2550 50  0000 C CNN
 F 1 "2.2K" V 3400 2550 50  0000 C CNN
-F 2 "" V 3330 2550 50  0001 C CNN
+F 2 "Resistors_SMD:R_0805" V 3330 2550 50  0001 C CNN
 F 3 "" H 3400 2550 50  0001 C CNN
 	1    3400 2550
@@
 F 0 "R5" V 4330 2300 50  0000 C CNN
 F 1 "100K" V 4250 2300 50  0000 C CNN
-F 2 "" V 4180 2300 50  0001 C CNN
+F 2 "Resistors_SMD:R_0603_HandSoldering" V 4180 2300 50  0001 C CNN
 F 3 "" H 4250 2300 50  0001 C CNN
 	1    4250 2300
@@
 F 0 "R6" V 4330 2700 50  0000 C CNN
 F 1 "100K" V 4250 2700 50  0000 C CNN
-F 2 "" V 4180 2700 50  0001 C CNN
+F 2 "Resistors_SMD:R_0603_HandSoldering" V 4180 2700 50  0001 C CNN
 F 3 "" H 4250 2700 50  0001 C CNN
 	1    4250 2700
@@
 F 0 "J10" H 2650 3600 50  0000 C CNN
 F 1 "I2C" H 2650 3200 50  0000 C CNN
-F 2 "" H 2650 3400 50  0001 C CNN
+F 2 "Pin_Headers:Pin_Header_Straight_1x03_Pitch2.54mm" H 2650 3400 50  0001 C CNN
 F 3 "" H 2650 3400 50  0001 C CNN
 	1    2650 3400
@@
 F 0 "J11" H 3400 3600 50  0000 C CNN
 F 1 "UART" H 3400 3200 50  0000 C CNN
-F 2 "" H 3400 3400 50  0001 C CNN
+F 2 "Pin_Headers:Pin_Header_Straight_1x03_Pitch2.54mm" H 3400 3400 50  0001 C CNN
 F 3 "" H 3400 3400 50  0001 C CNN
 	1    3400 3400
@@
 F 0 "R13" V 3980 1900 50  0000 C CNN
 F 1 "1k" V 3900 1900 50  0000 C CNN
-F 2 "" V 3830 1900 50  0001 C CNN
+F 2 "Resistors_SMD:R_0603_HandSoldering" V 3830 1900 50  0001 C CNN
 F 3 "" H 3900 1900 50  0001 C CNN
 	1    3900 1900
@@
 Wire Wire Line
 	3900 1350 3900 1450
+$Comp
+L GND #PWR067
+U 1 1 5B20802A
+P 1600 10600
+F 0 "#PWR067" H 1600 10350 50  0001 C CNN
+F 1 "GND" H 1600 10450 50  0000 C CNN
+F 2 "" H 1600 10600 50  0001 C CNN
+F 3 "" H 1600 10600 50  0001 C CNN
+	1    1600 10600
+	1    0    0    -1
+$EndComp
+Wire Wire Line
+	1600 10600 1600 10550
+Wire Wire Line
+	1600 10550 1750 10550
 $EndSCHEMATC
