File: Board3/_saved_AvionicsBoard.sch (KiCad schematic (older format))
At the start: 75 parts, among them J1 USB_A, J10 I2C, J11 UART, J12 RF IN, J13 RFD900 Connector, J2 Conn_01x02, J3 SWD, J4 7.2V, J5 SPI, J6 Micro_SD_Card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

Commit message: Add LEDs, cleanup traces
Parts:
- removed 1k, 1k? (x2): R, symbol R
- added R19, R20, R21: 1K, Resistors_SMD:R_0805, symbol R
- D4, D5, D6: renamed from D?; footprint (none) -> LEDs:LED_1206
Changed lines of the file:
@@
 D10
 $Comp
-L LED D?
+L LED D4
 U 1 1 5BDD1B4D
 P 9300 7300
-F 0 "D?" H 9300 7400 50  0000 C CNN
+F 0 "D4" H 9300 7400 50  0000 C CNN
 F 1 "LED" H 9300 7200 50  0000 C CNN
-F 2 "" H 9300 7300 50  0001 C CNN
+F 2 "LEDs:LED_1206" H 9300 7300 50  0001 C CNN
 F 3 "" H 9300 7300 50  0001 C CNN
 	1    9300 7300
@@
 $EndComp
 $Comp
-L R 1k
-U 1 1 5BDD20E2
-P 9600 7300
-F 0 "1k" V 9680 7300 50  0000 C CNN
-F 1 "R" V 9600 7300 50  0000 C CNN
-F 2 "" V 9530 7300 50  0001 C CNN
-F 3 "" H 9600 7300 50  0001 C CNN
-	1    9600 7300
-	0    1    1    0
-$EndComp
-$Comp
-L LED D?
+L LED D5
 U 1 1 5BDD4B11
 P 9300 7600
-F 0 "D?" H 9300 7700 50  0000 C CNN
+F 0 "D5" H 9300 7700 50  0000 C CNN
 F 1 "LED" H 9300 7500 50  0000 C CNN
-F 2 "" H 9300 7600 50  0001 C CNN
+F 2 "LEDs:LED_1206" H 9300 7600 50  0001 C CNN
 F 3 "" H 9300 7600 50  0001 C CNN
 	1    9300 7600
@@
 $EndComp
 $Comp
-L R 1k?
-U 1 1 5BDD4B17
-P 9600 7600
-F 0 "1k?" V 9680 7600 50  0000 C CNN
-F 1 "R" V 9600 7600 50  0000 C CNN
-F 2 "" V 9530 7600 50  0001 C CNN
-F 3 "" H 9600 7600 50  0001 C CNN
-	1    9600 7600
-	0    1    1    0
-$EndComp
-$Comp
-L LED D?
+L LED D6
 U 1 1 5BDD4BD1
 P 9300 7900
-F 0 "D?" H 9300 8000 50  0000 C CNN
+F 0 "D6" H 9300 8000 50  0000 C CNN
 F 1 "LED" H 9300 7800 50  0000 C CNN
-F 2 "" H 9300 7900 50  0001 C CNN
+F 2 "LEDs:LED_1206" H 9300 7900 50  0001 C CNN
 F 3 "" H 9300 7900 50  0001 C CNN
 	1    9300 7900
 	-1   0    0    1
-$EndComp
-$Comp
-L R 1k?
-U 1 1 5BDD4BD7
-P 9600 7900
-F 0 "1k?" V 9680 7900 50  0000 C CNN
-F 1 "R" V 9600 7900 50  0000 C CNN
-F 2 "" V 9530 7900 50  0001 C CNN
-F 3 "" H 9600 7900 50  0001 C CNN
-	1    9600 7900
-	0    1    1    0
 $EndComp
 Text Label 9150 7300 2    60   ~ 0
@@
 D12
 $Comp
-L GND #PWR?
+L GND #PWR082
 U 1 1 5BDD7E94
 P 9850 8100
-F 0 "#PWR?" H 9850 7850 50  0001 C CNN
+F 0 "#PWR082" H 9850 7850 50  0001 C CNN
 F 1 "GND" H 9850 7950 50  0000 C CNN
 F 2 "" H 9850 8100 50  0001 C CNN
@@
 	9750 7300 9850 7300
 Connection ~ 9850 7600
+$Comp
+L R R19
+U 1 1 5BDD8D3B
+P 9600 7300
+F 0 "R19" V 9680 7300 50  0000 C CNN
+F 1 "1K" V 9600 7300 50  0000 C CNN
+F 2 "Resistors_SMD:R_0805" V 9530 7300 50  0001 C CNN
+F 3 "" H 9600 7300 50  0001 C CNN
+	1    9600 7300
+	0    1    1    0
+$EndComp
+$Comp
+L R R20
+U 1 1 5BDD91DC
+P 9600 7600
+F 0 "R20" V 9680 7600 50  0000 C CNN
+F 1 "1K" V 9600 7600 50  0000 C CNN
+F 2 "Resistors_SMD:R_0805" V 9530 7600 50  0001 C CNN
+F 3 "" H 9600 7600 50  0001 C CNN
+	1    9600 7600
+	0    1    1    0
+$EndComp
+$Comp
+L R R21
+U 1 1 5BDD92DE
+P 9600 7900
+F 0 "R21" V 9680 7900 50  0000 C CNN
+F 1 "1K" V 9600 7900 50  0000 C CNN
+F 2 "Resistors_SMD:R_0805" V 9530 7900 50  0001 C CNN
+F 3 "" H 9600 7900 50  0001 C CNN
+	1    9600 7900
+	0    1    1    0
+$EndComp
 $EndSCHEMATC

Commit message: Added finshing touches to board. Investigate GPS and RFM95 RF paths!! RFD900 mounting hole sneed resizing!!
Parts:
- J12, J7: footprint Connectors:SMA_SMD_Jack_Straight -> FoxWestern:Edge_SMA
Changed lines of the file:
@@
 F 0 "J7" H 7810 1870 50  0000 C CNN
 F 1 "RF IN" V 7915 1750 50  0000 C CNN
-F 2 "Connectors:SMA_SMD_Jack_Straight" H 7800 1750 50  0001 C CNN
+F 2 "FoxWestern:Edge_SMA" H 7800 1750 50  0001 C CNN
 F 3 "" H 7800 1750 50  0001 C CNN
 	1    7800 1750
@@
 F 0 "J12" H 3660 10670 50  0000 C CNN
 F 1 "RF IN" V 3765 10550 50  0000 C CNN
-F 2 "Connectors:SMA_SMD_Jack_Straight" H 3650 10550 50  0001 C CNN
+F 2 "FoxWestern:Edge_SMA" H 3650 10550 50  0001 C CNN
 F 3 "" H 3650 10550 50  0001 C CNN
 	1    3650 10550
