File: Board3/_autosave-AvionicsBoard.kicad_pcb (KiCad board)
At the start: 2 copper layers, 101.7 x 53.2 mm, 61 parts, among them J1 USB_A, J10 I2C, J11 UART, J12 900MHz_Ant, J2 Conn_01x02, J5 SPI, J6 Micro_SD_Card, J7 RF IN, U1 TL1963, U10 ECS-.327-12.5-17X-TR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

Commit message: Finished routing board, added logo
Parts:
- added G***: LOGO, ManifestLabsLogo:Manifestabs, B.Cu at (109.7, 78.0)
Other:
- board text added: "Danny Mallek 2018"
