File: Board3/AvionicsBoard.kicad_pcb (KiCad board)
At the start: 2 copper layers, 157.4 x 59 mm, 85 parts, among them J1 USB_A, J11 UART, J12 RF IN, J13 RFD900 Connector, J2 Conn_01x02, J6 Micro_SD_Card, J7 RF IN, U1 TL1963, U10 ECS-.327-12.5-17X-TR, U11 GT-U7_GPS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

Commit message: Doen
Parts:
- removed the G*** at (111.8, 111.8)
- added G***: LOGO, RocketShopLogos:thumbsup, B.Cu at (111.9, 106.3)
- J12, J7: footprint FoxWestern:Edge_SMA -> FoxWestern:SMA_TH
- moved J12 15.0 mm to (198.6, 101.6), turned to 0 degrees
- moved J7 3.42 mm to (210.3, 93.0), turned to 0 degrees
Routing:
- net Net-(J12-Pad1): track 67.7 -> 52.0 mm
- net Net-(J7-Pad1): track 95.3 -> 93.6 mm
