File: Board4/AvionicsBoard.sch (KiCad schematic (older format))
At the start: 69 parts, among them J1 USB_A, J10 I2C, J11 UART, J12 RF IN, J13 RFD900 Connector, J2 Conn_01x02, J3 SWD, J4 7.2V, J5 SPI, J6 Micro_SD_Card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

Commit message: Change CS for SD card to PA08 (aka pin 13), Add RDF900 Serial ports, Add 0 ohm GPS selectors, add GT-07 GPS, add 5v regualtor for RFD900
Parts:
- removed C20, C21: 10u, Capacitors_SMD:C_1206, symbol C
- removed J13: RFD900 Connector, FoxWestern:RFD900, symbol Conn_02x08_Odd_Even
- removed R14, R15, R16, R17, R18: 0, Resistors_SMD:R_0805, symbol R
- removed U11: GT-U7_GPS, FoxWestern:GPS_GT-07, symbol GT-U7_GPS
- removed U12: LM340MP-5.0, TO_SOT_Packages_SMD:SOT-223-3_TabPin2, symbol LM340MP-5.0
- R1, R13, R5, R6: footprint Resistors_SMD:R_0805 -> Resistors_SMD:R_0603_HandSoldering
Connections:
- net labels added: CS
- net labels removed: +5V, RADIO_CS, RFD900_RX, RFD900_TX, SD_CS
- wire segments 183 -> 156
- no-connect marks 48 -> 37
