File: Board3 - Shorty/AvionicsBoard.sch (KiCad schematic (older format))
At the start: 59 parts, among them J1 USB_A, J10 I2C, J11 UART, J12 RF IN, J2 Conn_01x02, J3 SWD, J4 7.2V, J5 SPI, J6 Micro_SD_Card, J7 RF IN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

Commit message: Layout
Parts:
- removed F1: Fuse, Capacitors_SMD:C_1206, symbol Fuse
- BT1: footprint Battery_Holders:Keystone_1058_1x2032-CoinCell -> DannysLib:BR-1225A_HB
Connections:
- wire segments 151 -> 146
Other:
- moved on the sheet: BT1
Changed lines of the file:
@@
 LIBS:valves
 LIBS:FoxWestern
-LIBS:AvionicsBoard-cache
 EELAYER 25 0
 EELAYER END
@@
 L Battery_Cell BT1
 U 1 1 5B212EC3
-P 8900 6900
-F 0 "BT1" H 9000 7000 50  0000 L CNN
-F 1 "Battery_Cell" H 9000 6900 50  0000 L CNN
-F 2 "Battery_Holders:Keystone_1058_1x2032-CoinCell" V 8900 6960 50  0001 C CNN
-F 3 "" V 8900 6960 50  0001 C CNN
-	1    8900 6900
+P 10400 1800
+F 0 "BT1" H 10500 1900 50  0000 L CNN
+F 1 "Battery_Cell" H 10500 1800 50  0000 L CNN
+F 2 "DannysLib:BR-1225A_HB" V 10400 1860 50  0001 C CNN
+F 3 "" V 10400 1860 50  0001 C CNN
+	1    10400 1800
 	1    0    0    -1
 $EndComp
@@
 L GND #PWR034
 U 1 1 5B2130E7
-P 8900 7100
-F 0 "#PWR034" H 8900 6850 50  0001 C CNN
-F 1 "GND" H 8900 6950 50  0000 C CNN
-F 2 "" H 8900 7100 50  0001 C CNN
-F 3 "" H 8900 7100 50  0001 C CNN
-	1    8900 7100
+P 10400 2000
+F 0 "#PWR034" H 10400 1750 50  0001 C CNN
+F 1 "GND" H 10400 1850 50  0000 C CNN
+F 2 "" H 10400 2000 50  0001 C CNN
+F 3 "" H 10400 2000 50  0001 C CNN
+	1    10400 2000
 	1    0    0    -1
 $EndComp
@@
 $EndComp
 $Comp
-L Fuse F1
-U 1 1 5B202E3F
-P 3050 1350
-F 0 "F1" V 3130 1350 50  0000 C CNN
-F 1 "Fuse" V 2975 1350 50  0000 C CNN
-F 2 "Capacitors_SMD:C_1206" V 2980 1350 50  0001 C CNN
-F 3 "" H 3050 1350 50  0001 C CNN
-	1    3050 1350
-	0    1    1    0
-$EndComp
-$Comp
 L D_Zener D1
 U 1 1 5B2214FD
@@
 	1    0    0    -1
 $EndComp
-Text Label 8900 6700 0    60   ~ 0
+Text Label 10400 1600 0    60   ~ 0
 B+
 Text Label 7250 1500 2    60   ~ 0
 B+
-Text Label 4150 8000 0    60   ~ 0
-MAX_M8_TX
-Text Label 4150 7900 0    60   ~ 0
-MAX_M8_RX
 $Comp
 L C C8
@@
 	900  2900 800  2900
 Wire Wire Line
-	3200 1350 3900 1350
+	2750 1350 3900 1350
 Connection ~ 3600 1350
 Connection ~ 3250 1350
 Wire Wire Line
-	2750 1350 2900 1350
-Wire Wire Line
 	1700 4100 1700 4200
 Wire Wire Line
@@
 Connection ~ 7000 6600
 Wire Wire Line
-	8900 6700 8550 6700
-Wire Wire Line
-	8900 7000 8900 7100
-Wire Wire Line
-	8550 6800 8700 6800
-Wire Wire Line
-	8700 6800 8700 7050
-Wire Wire Line
-	8700 7050 8900 7050
-Connection ~ 8900 7050
+	10400 1900 10400 2000
 Wire Wire Line
 	7250 1700 7250 1600
@@
 Wire Wire Line
 	2350 8700 2350 8450
-Wire Wire Line
-	3850 8000 4150 8000
-Wire Wire Line
-	3850 7900 4150 7900
 Wire Wire Line
 	2600 9550 2600 10350
@@
 Wire Wire Line
 	8900 1500 8900 1550
-Text Label 7250 1200 2    60   ~ 0
-MAX_M8_RX
-Text Label 7250 1100 2    60   ~ 0
-MAX_M8_TX
 $Comp
 L MPL3115A2 U6
@@
 Wire Wire Line
 	8900 1500 8600 1500
+Wire Wire Line
+	3850 7900 4150 7900
+Wire Wire Line
+	3850 8000 4150 8000
+Text Label 4150 7900 0    60   ~ 0
+MAX_M8_RX
+Text Label 4150 8000 0    60   ~ 0
+MAX_M8_TX
+Text Label 7250 1200 2    60   ~ 0
+TXD
+Text Label 7250 1100 2    60   ~ 0
+RXD
 $EndSCHEMATC

Commit message: Do some board cleanup, generate gerbs
Parts:
- J2: value Conn_01x02 -> XT-60
- J4: value 7.2V -> 12v
Connections:
- net +12V: now also J2.1 (Pin_1)
- net GND: now also J2.2 (Pin_2); no longer J2.1 (Pin_1)
- net SCL: no longer U4.17 (SCL)
- net SDA: no longer U4.16 (SDA)
- net VBUS: no longer J2.2 (Pin_2)
- no-connect marks 36 -> 38
Other:
- moved on the sheet: J2, J4

Commit message: Add buzzer, LorA interrupt and reset lines, fix issue with USB and battery power, reduce RF path lengths, add better microstrip matching for LoRa and GPS, create ALLPCB BOM
Parts:
- removed U1: TL1963, TO_SOT_Packages_SMD:SOT-223-3_TabPin2, symbol TL1963
- added BZ1: Buzzer, DannysLib:CUI_CMT-5023S-SMT, symbol Buzzer
- added C20, C21: 10u, Capacitors_SMD:C_1206, symbol C
- added R4: 330, Resistors_SMD:R_0805, symbol R
- added U1: LT1117CST-3.3#TRPBF, TO_SOT_Packages_SMD:SOT-223-3_TabPin2, symbol LT1117CST-3.3#TRPBF
- added U3: MCP1825S, TO_SOT_Packages_SMD:SOT-223-3_TabPin2, symbol MCP1825S
- C12: footprint Capacitors_SMD:C_1206 -> Capacitors_SMD:C_0805
Connections:
- net +3V3: now also C21.1, U1.2 (OUT), U3.3 (VOUT)
- net A4: now also U8.6 (RESET)
- net A5: now also R4.1
- net D8: now also U8.14 (DIO0)
- net GND: now also BZ1.2 (+), C20.2, C21.2, U1.1 (GND), U3.2 (GND)
- net VBUS: now also C20.1, U3.1 (VIN); no longer C4.1, D1.1 (K)
- new net: C4.1, D1.1 (K), U1.3 (IN)
- new net: BZ1.1 (-), R4.2
- no-connect marks 38 -> 36
Other:
- note added: "Technically, there should be a PFET to switch off battery power\nand turn on USB power when the USB is plugged in, instead of two regulators.\nThis will be changed in the next revision."

Commit message: dsfafdsa
Parts:
- added C22: 100n, Capacitors_SMD:C_0805, symbol C
- added J13: SD_CS, Pin_Headers:Pin_Header_Straight_1x01_Pitch2.54mm, symbol Conn_01x01
- added J14: CHASSIS LED, Pin_Headers:Pin_Header_Straight_1x01_Pitch2.54mm, symbol Conn_01x01
- added J15, J16, J17, J18: CHASSIS GND, Mounting_Holes:MountingHole_2.5mm_Pad, symbol Conn_01x01
- C12: value 1u -> 10u
- C14: value .1u -> 100n
- J12, J7: footprint FoxWestern:SMA_TH -> DannysLib:SMA_TH
- U10, U9: footprint FoxWestern:XC1195CT-ND -> DannysLib:XC1195CT-ND
- U6: footprint FoxWestern:MPL3115A2 -> DannysLib:MPL3115A2
- U7: footprint FoxWestern:BNO055-LGA -> DannysLib:BNO055-LGA
- U8: footprint FoxWestern:RFM95W -> DannysLib:RFM95W
Connections:
- net +3V3: now also C22.1
- net D4: now also J13.1 (Pin_1)
- net D7: now also J14.1 (Pin_1)
- net GND: now also J6.9 (SHIELD), U5.13 (GND), C22.2, J15.1 (Pin_1), J16.1 (Pin_1), J17.1 (Pin_1), J18.1 (Pin_1)
- no-connect marks 36 -> 37
Other:
- moved on the sheet: C12, C14
Changed lines of the file:
@@
 F 0 "U7" H 12900 5750 60  0000 C CNN
 F 1 "BNO055" H 11850 6450 60  0000 C CNN
-F 2 "FoxWestern:BNO055-LGA" H 12600 5850 60  0001 C CNN
+F 2 "DannysLib:BNO055-LGA" H 12600 5850 60  0001 C CNN
 F 3 "" H 12600 5850 60  0001 C CNN
 	1    12600 5850
@@
 L C C14
 U 1 1 5B20EA08
-P 12050 1950
-F 0 "C14" H 12075 2050 50  0000 L CNN
-F 1 ".1u" H 12075 1850 50  0000 L CNN
-F 2 "Capacitors_SMD:C_0805" H 12088 1800 50  0001 C CNN
-F 3 "" H 12050 1950 50  0001 C CNN
-	1    12050 1950
+P 12050 1900
+F 0 "C14" H 12075 2000 50  0000 L CNN
+F 1 "100n" H 12075 1800 50  0000 L CNN
+F 2 "Capacitors_SMD:C_0805" H 12088 1750 50  0001 C CNN
+F 3 "" H 12050 1900 50  0001 C CNN
+	1    12050 1900
 	1    0    0    -1
 $EndComp
@@
 L C C12
 U 1 1 5B20EAC0
-P 11750 1950
-F 0 "C12" H 11775 2050 50  0000 L CNN
-F 1 "1u" H 11775 1850 50  0000 L CNN
-F 2 "Capacitors_SMD:C_0805" H 11788 1800 50  0001 C CNN
-F 3 "" H 11750 1950 50  0001 C CNN
-	1    11750 1950
+P 11750 1900
+F 0 "C12" H 11775 2000 50  0000 L CNN
+F 1 "10u" H 11775 1800 50  0000 L CNN
+F 2 "Capacitors_SMD:C_0805" H 11788 1750 50  0001 C CNN
+F 3 "" H 11750 1900 50  0001 C CNN
+	1    11750 1900
 	1    0    0    -1
 $EndComp
@@
 L +3.3V #PWR030
 U 1 1 5B20EEA4
-P 11750 1600
-F 0 "#PWR030" H 11750 1450 50  0001 C CNN
-F 1 "+3.3V" H 11750 1740 50  0000 C CNN
-F 2 "" H 11750 1600 50  0001 C CNN
-F 3 "" H 11750 1600 50  0001 C CNN
-	1    11750 1600
+P 11450 1550
+F 0 "#PWR030" H 11450 1400 50  0001 C CNN
+F 1 "+3.3V" H 11450 1690 50  0000 C CNN
+F 2 "" H 11450 1550 50  0001 C CNN
+F 3 "" H 11450 1550 50  0001 C CNN
+	1    11450 1550
 	1    0    0    -1
 $EndComp
@@
 F 0 "J7" H 9310 1970 50  0000 C CNN
 F 1 "RF IN" V 9415 1850 50  0000 C CNN
-F 2 "FoxWestern:SMA_TH" H 9300 1850 50  0001 C CNN
+F 2 "DannysLib:SMA_TH" H 9300 1850 50  0001 C CNN
 F 3 "" H 9300 1850 50  0001 C CNN
 	1    9300 1850
@@
 F 0 "U9" V 900 4750 60  0000 C CNN
 F 1 "ECS-.327-12.5-17X-TR" V 1200 5050 60  0000 C CNN
-F 2 "FoxWestern:XC1195CT-ND" H 1150 5000 60  0001 C CNN
+F 2 "DannysLib:XC1195CT-ND" H 1150 5000 60  0001 C CNN
 F 3 "" H 1150 5000 60  0001 C CNN
 	1    1150 5000
@@
 F 0 "U10" V 13600 3550 60  0000 C CNN
 F 1 "ECS-.327-12.5-17X-TR" V 13900 3850 60  0000 C CNN
-F 2 "FoxWestern:XC1195CT-ND" H 13850 3800 60  0001 C CNN
+F 2 "DannysLib:XC1195CT-ND" H 13850 3800 60  0001 C CNN
 F 3 "" H 13850 3800 60  0001 C CNN
 	1    13850 3800
@@
 F 0 "J12" H 9310 4320 50  0000 C CNN
 F 1 "RF IN" V 9415 4200 50  0000 C CNN
-F 2 "FoxWestern:SMA_TH" H 9300 4200 50  0001 C CNN
+F 2 "DannysLib:SMA_TH" H 9300 4200 50  0001 C CNN
 F 3 "" H 9300 4200 50  0001 C CNN
 	1    9300 4200
@@
 F 0 "U6" H 13300 1500 60  0000 C CNN
 F 1 "MPL3115A2" H 13050 2000 60  0000 C CNN
-F 2 "FoxWestern:MPL3115A2" H 13050 1350 60  0001 C CNN
+F 2 "DannysLib:MPL3115A2" H 13050 1350 60  0001 C CNN
 F 3 "" H 13050 1350 60  0001 C CNN
 	1    13050 1750
@@
 	1700 4400 1700 4450
 Wire Wire Line
-	12050 1800 12050 1700
+	12050 1750 12050 1700
 Wire Wire Line
 	12050 1700 12550 1700
 Wire Wire Line
-	11750 1600 12550 1600
-Wire Wire Line
-	11750 1600 11750 1800
-Wire Wire Line
-	11750 2150 12250 2150
-Wire Wire Line
-	11750 2150 11750 2100
-Wire Wire Line
-	12050 2150 12050 2100
+	11450 1600 12550 1600
+Wire Wire Line
+	11750 1600 11750 1750
+Wire Wire Line
+	11450 2150 12250 2150
+Wire Wire Line
+	11750 2150 11750 2050
+Wire Wire Line
+	12050 2150 12050 2050
 Connection ~ 11900 2150
 Wire Wire Line
@@
 F 0 "U8" H 8250 3400 60  0000 C CNN
 F 1 "RFM95W" H 7950 4300 60  0000 C CNN
-F 2 "FoxWestern:RFM95W" H 7950 3850 60  0001 C CNN
+F 2 "DannysLib:RFM95W" H 7950 3850 60  0001 C CNN
 F 3 "" H 7950 3850 60  0001 C CNN
 	1    7950 3850
@@
 Text Notes 4250 2750 0    60   ~ 0
 Technically, there should be a PFET to switch off battery power\nand turn on USB power when the USB is plugged in, instead of two regulators.\nThis will be changed in the next revision.
+$Comp
+L Conn_01x01 J13
+U 1 1 5C32936E
+P 5900 10250
+F 0 "J13" H 5900 10350 50  0000 C CNN
+F 1 "SD_CS" H 5900 10150 50  0000 C CNN
+F 2 "Pin_Headers:Pin_Header_Straight_1x01_Pitch2.54mm" H 5900 10250 50  0001 C CNN
+F 3 "" H 5900 10250 50  0001 C CNN
+	1    5900 10250
+	1    0    0    -1
+$EndComp
+Text Label 5700 10250 2    60   ~ 0
+SD_CS
+$Comp
+L C C22
+U 1 1 5C32A6AF
+P 11450 1900
+F 0 "C22" H 11475 2000 50  0000 L CNN
+F 1 "100n" H 11475 1800 50  0000 L CNN
+F 2 "Capacitors_SMD:C_0805" H 11488 1750 50  0001 C CNN
+F 3 "" H 11450 1900 50  0001 C CNN
+	1    11450 1900
+	1    0    0    -1
+$EndComp
+Wire Wire Line
+	11450 2150 11450 2050
+Connection ~ 11750 2150
+Wire Wire Line
+	11450 1550 11450 1750
+Connection ~ 11750 1600
+Connection ~ 11450 1600
+$Comp
+L Conn_01x01 J14
+U 1 1 5C32E2A4
+P 2250 9250
+F 0 "J14" H 2250 9350 50  0000 C CNN
+F 1 "CHASSIS LED" H 2250 9150 50  0000 C CNN
+F 2 "Pin_Headers:Pin_Header_Straight_1x01_Pitch2.54mm" H 2250 9250 50  0001 C CNN
+F 3 "" H 2250 9250 50  0001 C CNN
+	1    2250 9250
+	1    0    0    -1
+$EndComp
+Wire Wire Line
+	1900 9550 1900 9250
+Wire Wire Line
+	1900 9250 2050 9250
+$Comp
+L GND #PWR075
+U 1 1 5C330EF1
+P 8750 6850
+F 0 "#PWR075" H 8750 6600 50  0001 C CNN
+F 1 "GND" H 8750 6700 50  0000 C CNN
+F 2 "" H 8750 6850 50  0001 C CNN
+F 3 "" H 8750 6850 50  0001 C CNN
+	1    8750 6850
+	1    0    0    -1
+$EndComp
+Wire Wire Line
+	8750 6850 8750 6800
+Wire Wire Line
+	8750 6800 8550 6800
+NoConn ~ 8550 6700
+$Comp
+L Conn_01x01 J15
+U 1 1 5C331C30
+P 12700 8200
+F 0 "J15" H 12700 8300 50  0000 C CNN
+F 1 "CHASSIS GND" H 12700 8100 50  0000 C CNN
+F 2 "Mounting_Holes:MountingHole_2.5mm_Pad" H 12700 8200 50  0001 C CNN
+F 3 "" H 12700 8200 50  0001 C CNN
+	1    12700 8200
+	1    0    0    -1
+$EndComp
+$Comp
+L GND #PWR076
+U 1 1 5C3325F2
+P 12400 9200
+F 0 "#PWR076" H 12400 8950 50  0001 C CNN
+F 1 "GND" H 12400 9050 50  0000 C CNN
+F 2 "" H 12400 9200 50  0001 C CNN
+F 3 "" H 12400 9200 50  0001 C CNN
+	1    12400 9200
+	1    0    0    -1
+$EndComp
+$Comp
+L Conn_01x01 J16
+U 1 1 5C332796
+P 12700 8500
+F 0 "J16" H 12700 8600 50  0000 C CNN
+F 1 "CHASSIS GND" H 12700 8400 50  0000 C CNN
+F 2 "Mounting_Holes:MountingHole_2.5mm_Pad" H 12700 8500 50  0001 C CNN
+F 3 "" H 12700 8500 50  0001 C CNN
+	1    12700 8500
+	1    0    0    -1
+$EndComp
+$Comp
+L Conn_01x01 J17
+U 1 1 5C33287E
+P 12700 8800
+F 0 "J17" H 12700 8900 50  0000 C CNN
+F 1 "CHASSIS GND" H 12700 8700 50  0000 C CNN
+F 2 "Mounting_Holes:MountingHole_2.5mm_Pad" H 12700 8800 50  0001 C CNN
+F 3 "" H 12700 8800 50  0001 C CNN
+	1    12700 8800
+	1    0    0    -1
+$EndComp
+$Comp
+L Conn_01x01 J18
+U 1 1 5C332973
+P 12700 9100
+F 0 "J18" H 12700 9200 50  0000 C CNN
+F 1 "CHASSIS GND" H 12700 9000 50  0000 C CNN
+F 2 "Mounting_Holes:MountingHole_2.5mm_Pad" H 12700 9100 50  0001 C CNN
+F 3 "" H 12700 9100 50  0001 C CNN
+	1    12700 9100
+	1    0    0    -1
+$EndComp
+Wire Wire Line
+	12400 8200 12400 9200
+Wire Wire Line
+	12400 9100 12500 9100
+Wire Wire Line
+	12400 8800 12500 8800
+Connection ~ 12400 9100
+Wire Wire Line
+	12400 8500 12500 8500
+Connection ~ 12400 8800
+Wire Wire Line
+	12400 8200 12500 8200
+Connection ~ 12400 8500
+$Comp
+L GND #PWR?
+U 1 1 5C335F34
+P 9050 10200
+F 0 "#PWR?" H 9050 9950 50  0001 C CNN
+F 1 "GND" H 9050 10050 50  0000 C CNN
+F 2 "" H 9050 10200 50  0001 C CNN
+F 3 "" H 9050 10200 50  0001 C CNN
+	1    9050 10200
+	1    0    0    -1
+$EndComp
+Wire Wire Line
+	9050 10200 9050 10150
+Wire Wire Line
+	9050 10150 9000 10150
 $EndSCHEMATC
