File: Test Rocket Avionics/Boards/Avionics Board 1/_autosave-Avionics Board 1.kicad_pcb (KiCad board)
At the start: 4 copper layers, 50 x 50 mm, 71 parts, among them J1 USB_A, J14 1S LiPo, J2 1S LiPo, J3 EXPANSION_HEADER, J4 USB_A, J5 SERVO, M2.5 CHASSIS_GND, U1 ECS-.327-12.5-17X-TR, U10 NC7WZ07, U11 LMR62014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

Commit message: Remove DS3231
Parts:
- removed C21: 1u, Capacitors_SMD:C_0805
- removed R10, R11: 10k, Resistors_SMD:R_0805
- removed U6: DS3231-SO16, Housings_SOIC:SOIC-16W_7.5x10.3mm_Pitch1.27mm
- C22: renamed from C14; moved to B.Cu
- moved C22 12.8 mm to (49.2, 114.5), turned to 90 degrees
- renumbered M2.5 to J10, M2.5 to J11, M2.5 to J12, M2.5 to J13
Connections:
- C22 pad 1: Net-(C14-Pad1) -> Net-(C22-Pad1)
Routing:
- net Net-(R11-Pad1): track 10.2 -> 0.00 mm
- net +3V3: track 75.0 -> 67.1 mm, vias 16 -> 13
- net /6V_SERVO_SUPPLY: track 18.1 -> 22.8 mm
- net Net-(C22-Pad1): track 7.41 -> 11.8 mm
- net Net-(R10-Pad1): track 3.66 -> 0.00 mm
- net Net-(C14-Pad1): track 1.54 -> 0.00 mm, vias 1 -> 0
- net GND: track 110.0 -> 108.5 mm, vias 35 -> 34
Other:
- outline, holes or cut-outs redrawn
