File: Test Rocket Avionics/Boards/Avionics Board 1/_saved_Avionics Board 1.sch (KiCad schematic (older format))
At the start: 65 parts, among them J1 USB_A, J10 CHASSIS_GND, J11 CHASSIS_GND, J12 CHASSIS_GND, J13 CHASSIS_GND, J14 1S LiPo, J2 1S LiPo, J3 EXPANSION_HEADER, J4 USB_A, J5 SERVO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

Commit message: Add micro SD Card, clean up ref des, power 6v boost directly from battery instead of 3.3V rail
Connections:
- net +3V3: no longer C20.1, L1.2, R17.1, U11.5 (VIN)
- net +BATT: now also C20.1, L1.2, R17.1, U11.5 (VIN)
- net GND: now also J6.9 (SHIELD)
Changed lines of the file:
@@
-$EndComp
-$Comp
-L Avionics-Board-1-rescue:+3.3V #PWR053
-U 1 1 5C726425
-P 12700 1300
-F 0 "#PWR053" H 12700 1150 50  0001 C CNN
-F 1 "+3.3V" H 12700 1440 50  0000 C CNN
-F 2 "" H 12700 1300 50  0001 C CNN
-F 3 "" H 12700 1300 50  0001 C CNN
-	1    12700 1300
-	1    0    0    -1
 $EndComp
 $Comp
@@
 Wire Wire Line
 	12300 1400 12400 1400
-Wire Wire Line
-	12700 1300 12700 1400
 Connection ~ 12700 1400
 $Comp
@@
 Wire Wire Line
 	7650 9300 8100 9300
+$Comp
+L Avionics-Board-1-rescue:GND #PWR0101
+U 1 1 5CCE34EA
+P 9900 9850
+F 0 "#PWR0101" H 9900 9600 50  0001 C CNN
+F 1 "GND" H 9900 9700 50  0000 C CNN
+F 2 "" H 9900 9850 50  0001 C CNN
+F 3 "" H 9900 9850 50  0001 C CNN
+	1    9900 9850
+	1    0    0    -1
+$EndComp
+Wire Wire Line
+	9900 9700 9800 9700
+Wire Wire Line
+	9900 9700 9900 9850
+$Comp
+L Avionics-Board-1-rescue:+BATT #PWR0102
+U 1 1 5CDB5E96
+P 12700 1200
+F 0 "#PWR0102" H 12700 1050 50  0001 C CNN
+F 1 "+BATT" H 12700 1340 50  0000 C CNN
+F 2 "" H 12700 1200 50  0001 C CNN
+F 3 "" H 12700 1200 50  0001 C CNN
+	1    12700 1200
+	1    0    0    -1
+$EndComp
+Wire Wire Line
+	12700 1200 12700 1400
 $EndSCHEMATC
