File: Test Rocket Avionics/Boards/RF Board/RF Board.kicad_pcb (KiCad board)
At the start: 4 copper layers, 50 x 50 mm, 7 parts, among them J1 EXPANSION_HEADER, J10 CHASSIS_GND, J11 CHASSIS_GND, J12 CHASSIS_GND, J13 CHASSIS_GND

Commit message: Mostly create RF Board
Parts:
- added C1: 10u, Capacitors_SMD:C_0805, F.Cu at (46.4, 125.4)
- added C2: 1u, Capacitors_SMD:C_0805, F.Cu at (51.0, 125.3)
- added C3: 10n, Capacitors_SMD:C_0805, F.Cu at (43.3, 110.6)
- added J2: LoRa, DannysLib:SMA_TH, F.Cu at (38.3, 103.5)
- added J3: GPS, DannysLib:SMA_TH, F.Cu at (52.0, 108.3)
- added R1: 10, Resistors_SMD:R_0805, F.Cu at (45.7, 110.7)
- added U1: RFM95W, DannysLib:RFM95W, F.Cu at (52.3, 82.1)
- added U2: MAX-M8, DannysLib:MAX_M82, F.Cu at (52.2, 114.1)
- moved G*** 8.89 mm to (43.7, 93.2)
- moved G*** 2.52 mm to (41.9, 106.8)
Routing:
- net /SCK: track 0.00 -> 62.6 mm, vias 0 -> 1
- net /MISO: track 0.00 -> 62.1 mm, vias 0 -> 1
- net /MOSI: track 0.00 -> 57.4 mm, vias 0 -> 1
- net +3V3: track 0.00 -> 45.2 mm, vias 0 -> 3
- net /RADIO_CS: track 0.00 -> 40.9 mm, vias 0 -> 1
- net /LORA_RESET: track 0.00 -> 39.0 mm, vias 0 -> 1
- net /LORA_INTERRUPT: track 0.00 -> 26.9 mm, vias 0 -> 1
- net /MAX_M8_TX: track 0.00 -> 22.4 mm, vias 0 -> 1
- net /MAX_M8_RX: track 0.00 -> 20.7 mm
- net Net-(C3-Pad1): track 0.00 -> 7.86 mm
- net GND: track 1.58 -> 7.75 mm
- net Net-(R1-Pad2): track 0.00 -> 2.86 mm
- net Net-(J3-Pad1): track 0.00 -> 1.10 mm
- added copper zone on F.Cu, net GND
