File: Test Rocket Avionics/Boards/RF Board/RF Board.sch (KiCad schematic (older format))
At the start: 5 parts, among them J1 EXPANSION_HEADER, J10 CHASSIS_GND, J11 CHASSIS_GND, J12 CHASSIS_GND, J13 CHASSIS_GND

Commit message: Mostly create RF Board
Parts:
- added C1: 10u, Capacitors_SMD:C_0805, symbol Device:C
- added C2: 1u, Capacitors_SMD:C_0805, symbol Device:C
- added C3: 10n, Capacitors_SMD:C_0805, symbol Device:C
- added J2: LoRa, DannysLib:SMA_TH, symbol Connector:Conn_Coaxial
- added J3: GPS, DannysLib:SMA_TH, symbol Connector:Conn_Coaxial
- added R1: 10, Resistors_SMD:R_0805, symbol Device:R
- added U1: RFM95W, DannysLib:RFM95W, symbol Danny's_Lib:RFM95W
- added U2: MAX-M8, DannysLib:MAX_M82, symbol Danny's_Lib:MAX-M8
Connections:
- net +3V3: now also C1.1, C2.1, U1.13 (3.3V), U2.13 (LNA_EN), U2.6 (V_BCKP), U2.7 (VCC_IO), U2.8 (VCC)
- net GND: now also C1.2, C2.2, C3.2, J2.2 (Ext), J3.2 (Ext), U1.1 (GND), U1.10 (GND), U1.8 (GND), U2.1 (GND), U2.10 (GND), U2.12 (GND)
- net LORA_INTERRUPT: now also U1.14 (DIO0)
- net LORA_RESET: now also U1.6 (RESET)
- net MAX_M8_RX: now also U2.2 (TXD)
- net MAX_M8_TX: now also U2.3 (RXD)
- net MISO: now also U1.2 (MISO)
- net MOSI: now also U1.3 (MOSI)
- net RADIO_CS: now also U1.5 (NSS)
- net SCK: now also U1.4 (SCK)
- new net: J2.1 (In), U1.9 (ANT)
- new net: J3.1 (In), U2.11 (RF_IN)
- new net: C3.1, R1.1, U2.14 (VCC_RF)
- new net: R1.2, U2.15 (V_ANT)
- no-connect marks 0 -> 11
